Commit message: Update arm urdf.

File: interbotix_ros_xsarms/interbotix_xsarm_descriptions/urdf/doris_arm.urdf.xacro (robot description, xacro)
@@ -48,5 +48,5 @@
         <axis xyz="0 0 1"/>
         <limit effort="10" lower="${-pi + pi_offset}" upper="${pi - pi_offset}" velocity="${pi}"/>
-        <origin rpy="0 0 0" xyz="0 0 0.049"/>
+        <origin rpy="0 0 0" xyz="0 0 0.023"/>
         <parent link="$(arg robot_name)/$(arg base_link_frame)"/>
         <child link="$(arg robot_name)/shoulder_link"/>
@@ -64,5 +64,5 @@
     <link name="$(arg robot_name)/shoulder_link">
         <visual>
-            <origin rpy="0 0 0" xyz="0 0 -0.003"/>
+            <origin rpy="0 0 0" xyz="0 0 0"/>
             <geometry>
                 <mesh filename="package://interbotix_xsarm_descriptions/meshes/doris_arm_meshes/doris_arm_2_shoulder.stl" scale="0.001 0.001 0.001"/>
@@ -71,5 +71,5 @@
         </visual>
         <collision>
-            <origin rpy="0 0 0" xyz="0 0 -0.003"/>
+            <origin rpy="0 0 0" xyz="0 0 0"/>
             <geometry>
                 <mesh filename="package://interbotix_xsarm_descriptions/meshes/doris_arm_meshes/doris_arm_2_shoulder.stl" scale="0.001 0.001 0.001"/>
@@ -175,5 +175,5 @@
     <link name="$(arg robot_name)/wrist_link">
         <visual>
-            <origin rpy="0 0 ${pi/2}" xyz="0 0 0"/>
+            <origin rpy="0 0 ${pi}" xyz="0 0 0"/>
             <geometry>
                 <mesh filename="package://interbotix_xsarm_descriptions/meshes/doris_arm_meshes/doris_arm_5_wrist.stl" scale="0.001 0.001 0.001"/>
@@ -182,5 +182,5 @@
         </visual>
         <collision>
-            <origin rpy="0 0 ${pi/2}" xyz="0 0 0"/>
+            <origin rpy="0 0 ${pi}" xyz="0 0 0"/>
             <geometry>
                 <mesh filename="package://interbotix_xsarm_descriptions/meshes/doris_arm_meshes/doris_arm_5_wrist.stl" scale="0.001 0.001 0.001"/>
@@ -212,5 +212,5 @@
     <link name="$(arg robot_name)/gripper_link">
         <visual>
-            <origin rpy="0 0 ${pi/2}" xyz="-0.02 0 0"/>
+            <origin rpy="0 0 0" xyz="-0.02 0 0"/>
             <geometry>
                 <mesh filename="package://interbotix_xsarm_descriptions/meshes/doris_arm_meshes/doris_arm_6_gripper.stl" scale="0.001 0.001 0.001"/>
@@ -219,5 +219,5 @@
         </visual>
         <collision>
-            <origin rpy="0 0 ${pi/2}" xyz="-0.02 0 0"/>
+            <origin rpy="0 0 0" xyz="-0.02 0 0"/>
             <geometry>
                 <mesh filename="package://interbotix_xsarm_descriptions/meshes/doris_arm_meshes/doris_arm_6_gripper.stl" scale="0.001 0.001 0.001"/>
@@ -260,5 +260,5 @@
     </transmission>
     <link name="$(arg robot_name)/gripper_prop_link">
-        <visual>
+        <!--visual>
             <origin rpy="0 0 ${pi/2}" xyz="-0.0685 0 0"/>
             <geometry>
@@ -272,5 +272,5 @@
                 <mesh filename="package://interbotix_xsarm_descriptions/meshes/doris_arm_meshes/doris_arm_7_gripper_prop.stl" scale="0.001 0.001 0.001"/>
             </geometry>
-        </collision>
+        </collision-->
         <inertial>
             <origin rpy="0 0 ${pi/2}" xyz="0.0023780000 0.0000000285 0.0000000000"/>
@@ -317,5 +317,5 @@
         </joint>
         <link name="$(arg robot_name)/gripper_bar_link">
-            <visual>
+            <!--visual>
                 <origin rpy="0 0 ${pi/2}" xyz="-0.063 0 0"/>
                 <geometry>
@@ -329,5 +329,5 @@
                     <mesh filename="package://interbotix_xsarm_descriptions/meshes/doris_arm_meshes/doris_arm_8_gripper_bar.stl" scale="0.001 0.001 0.001"/>
                 </geometry>
-            </collision>
+            </collision-->
             <inertial>
                 <origin rpy="0 0 ${pi/2}" xyz="0.0067940000 -0.0000004272 -0.0007760000"/>
@@ -369,5 +369,5 @@
             <link name="$(arg robot_name)/left_finger_link">
                 <visual>
-                    <origin rpy="${pi/2} ${-pi} ${pi/2}" xyz="-0.0404 -0.0575 0"/>
+                    <origin rpy="${pi} 0 0" xyz="0 0 0"/>
                     <geometry>
                         <mesh filename="package://interbotix_xsarm_descriptions/meshes/doris_arm_meshes/doris_arm_9_gripper_finger.stl" scale="0.001 0.001 0.001"/>
@@ -376,5 +376,5 @@
                 </visual>
                 <collision>
-                    <origin rpy="${pi/2} ${-pi} ${pi/2}" xyz="-0.0404 -0.0575 0"/>
+                    <origin rpy="${pi} 0 0" xyz="0 0 0"/>
                     <geometry>
                         <mesh filename="package://interbotix_xsarm_descriptions/meshes/doris_arm_meshes/doris_arm_9_gripper_finger.stl" scale="0.001 0.001 0.001"/>
@@ -409,5 +409,5 @@
             <link name="$(arg robot_name)/right_finger_link">
                 <visual>
-                    <origin rpy="${-pi/2} ${pi} ${-pi/2}" xyz="-0.0404 0.0575 0 "/>
+                    <origin rpy="0 0 0" xyz="0 0 0 "/>
                     <geometry>
                         <mesh filename="package://interbotix_xsarm_descriptions/meshes/doris_arm_meshes/doris_arm_9_gripper_finger.stl" scale="0.001 0.001 0.001"/>
@@ -416,5 +416,5 @@
                 </visual>
                 <collision>
-                    <origin rpy="${-pi/2} ${pi} ${-pi/2}" xyz="-0.0404 0.0575 0 "/>
+                    <origin rpy="0 0 0" xyz="0 0 0 "/>
                     <geometry>
                         <mesh filename="package://interbotix_xsarm_descriptions/meshes/doris_arm_meshes/doris_arm_9_gripper_finger.stl" scale="0.001 0.001 0.001"/>

Commit message: Update arm urdf meshes

File: interbotix_ros_xsarms/interbotix_xsarm_descriptions/urdf/doris_arm.urdf.xacro (robot description, xacro)
@@ -29,12 +29,12 @@
             <origin rpy="0 0 0" xyz="0 0 0"/>
             <geometry>
-                <mesh filename="package://interbotix_xsarm_descriptions/meshes/doris_arm_meshes/doris_arm_1_base.stl" scale="0.001 0.001 0.001"/>
-            </geometry>
-            <material name="interbotix_black"/>
-        </visual>
-        <collision>
-            <origin rpy="0 0 0" xyz="0 0 0"/>
-            <geometry>
-                <mesh filename="package://interbotix_xsarm_descriptions/meshes/doris_arm_meshes/doris_arm_1_base.stl" scale="0.001 0.001 0.001"/>
+                <mesh filename="package://interbotix_xsarm_descriptions/meshes/doris_arm_meshes/doris_arm_1_base.stl" />
+            </geometry>
+            <material name="interbotix_black"/>
+        </visual>
+        <collision>
+            <origin rpy="0 0 0" xyz="0 0 0"/>
+            <geometry>
+                <mesh filename="package://interbotix_xsarm_descriptions/meshes/doris_arm_meshes/doris_arm_1_base.stl" />
             </geometry>
         </collision>
@@ -66,12 +66,12 @@
             <origin rpy="0 0 0" xyz="0 0 0"/>
             <geometry>
-                <mesh filename="package://interbotix_xsarm_descriptions/meshes/doris_arm_meshes/doris_arm_2_shoulder.stl" scale="0.001 0.001 0.001"/>
-            </geometry>
-            <material name="interbotix_black"/>
-        </visual>
-        <collision>
-            <origin rpy="0 0 0" xyz="0 0 0"/>
-            <geometry>
-                <mesh filename="package://interbotix_xsarm_descriptions/meshes/doris_arm_meshes/doris_arm_2_shoulder.stl" scale="0.001 0.001 0.001"/>
+                <mesh filename="package://interbotix_xsarm_descriptions/meshes/doris_arm_meshes/doris_arm_2_shoulder.stl" />
+            </geometry>
+            <material name="interbotix_black"/>
+        </visual>
+        <collision>
+            <origin rpy="0 0 0" xyz="0 0 0"/>
+            <geometry>
+                <mesh filename="package://interbotix_xsarm_descriptions/meshes/doris_arm_meshes/doris_arm_2_shoulder.stl" />
             </geometry>
         </collision>
@@ -103,12 +103,12 @@
             <origin rpy="0 0 0" xyz="0 0 0"/>
             <geometry>
-                <mesh filename="package://interbotix_xsarm_descriptions/meshes/doris_arm_meshes/doris_arm_3_upper_arm.stl" scale="0.001 0.001 0.001"/>
-            </geometry>
-            <material name="interbotix_black"/>
-        </visual>
-        <collision>
-            <origin rpy="0 0 0" xyz="0 0 0"/>
-            <geometry>
-                <mesh filename="package://interbotix_xsarm_descriptions/meshes/doris_arm_meshes/doris_arm_3_upper_arm.stl" scale="0.001 0.001 0.001"/>
+                <mesh filename="package://interbotix_xsarm_descriptions/meshes/doris_arm_meshes/doris_arm_3_upper_arm.stl" />
+            </geometry>
+            <material name="interbotix_black"/>
+        </visual>
+        <collision>
+            <origin rpy="0 0 0" xyz="0 0 0"/>
+            <geometry>
+                <mesh filename="package://interbotix_xsarm_descriptions/meshes/doris_arm_meshes/doris_arm_3_upper_arm.stl" />
             </geometry>
         </collision>
@@ -140,12 +140,12 @@
             <origin rpy="0 0 0" xyz="0 0 0"/>
             <geometry>
-                <mesh filename="package://interbotix_xsarm_descriptions/meshes/doris_arm_meshes/doris_arm_4_forearm.stl" scale="0.001 0.001 0.001"/>
-            </geometry>
-            <material name="interbotix_black"/>
-        </visual>
-        <collision>
-            <origin rpy="0 0 0" xyz="0 0 0"/>
-            <geometry>
-                <mesh filename="package://interbotix_xsarm_descriptions/meshes/doris_arm_meshes/doris_arm_4_forearm.stl" scale="0.001 0.001 0.001"/>
+                <mesh filename="package://interbotix_xsarm_descriptions/meshes/doris_arm_meshes/doris_arm_4_forearm.stl" />
+            </geometry>
+            <material name="interbotix_black"/>
+        </visual>
+        <collision>
+            <origin rpy="0 0 0" xyz="0 0 0"/>
+            <geometry>
+                <mesh filename="package://interbotix_xsarm_descriptions/meshes/doris_arm_meshes/doris_arm_4_forearm.stl" />
             </geometry>
         </collision>
@@ -177,5 +177,5 @@
             <origin rpy="0 0 ${pi}" xyz="0 0 0"/>
             <geometry>
-                <mesh filename="package://interbotix_xsarm_descriptions/meshes/doris_arm_meshes/doris_arm_5_wrist.stl" scale="0.001 0.001 0.001"/>
+                <mesh filename="package://interbotix_xsarm_descriptions/meshes/doris_arm_meshes/doris_arm_5_wrist.stl" />
             </geometry>
             <material name="interbotix_black"/>
@@ -184,5 +184,5 @@
             <origin rpy="0 0 ${pi}" xyz="0 0 0"/>
             <geometry>
-                <mesh filename="package://interbotix_xsarm_descriptions/meshes/doris_arm_meshes/doris_arm_5_wrist.stl" scale="0.001 0.001 0.001"/>
+                <mesh filename="package://interbotix_xsarm_descriptions/meshes/doris_arm_meshes/doris_arm_5_wrist.stl" />
             </geometry>
         </collision>
@@ -214,5 +214,5 @@
             <origin rpy="0 0 0" xyz="-0.02 0 0"/>
             <geometry>
-                <mesh filename="package://interbotix_xsarm_descriptions/meshes/doris_arm_meshes/doris_arm_6_gripper.stl" scale="0.001 0.001 0.001"/>
+                <mesh filename="package://interbotix_xsarm_descriptions/meshes/doris_arm_meshes/doris_arm_6_gripper.stl" />
             </geometry>
             <material name="interbotix_black"/>
@@ -221,5 +221,5 @@
             <origin rpy="0 0 0" xyz="-0.02 0 0"/>
             <geometry>
-                <mesh filename="package://interbotix_xsarm_descriptions/meshes/doris_arm_meshes/doris_arm_6_gripper.stl" scale="0.001 0.001 0.001"/>
+                <mesh filename="package://interbotix_xsarm_descriptions/meshes/doris_arm_meshes/doris_arm_6_gripper.stl" />
             </geometry>
         </collision>
@@ -263,5 +263,5 @@
             <origin rpy="0 0 ${pi/2}" xyz="-0.0685 0 0"/>
             <geometry>
-                <mesh filename="package://interbotix_xsarm_descriptions/meshes/doris_arm_meshes/doris_arm_7_gripper_prop.stl" scale="0.001 0.001 0.001"/>
+                <mesh filename="package://interbotix_xsarm_descriptions/meshes/doris_arm_meshes/doris_arm_7_gripper_prop.stl" />
             </geometry>
             <material name="interbotix_black"/>
@@ -270,5 +270,5 @@
             <origin rpy="0 0 ${pi/2}" xyz="-0.0685 0 0"/>
             <geometry>
-                <mesh filename="package://interbotix_xsarm_descriptions/meshes/doris_arm_meshes/doris_arm_7_gripper_prop.stl" scale="0.001 0.001 0.001"/>
+                <mesh filename="package://interbotix_xsarm_descriptions/meshes/doris_arm_meshes/doris_arm_7_gripper_prop.stl" />
             </geometry>
         </collision-->
@@ -291,5 +291,5 @@
                 <origin rpy="0 0 0" xyz="0 0 0"/>
                 <geometry>
-                    <mesh filename="package://interbotix_xsarm_descriptions/meshes/doris_arm_meshes/doris_arm_10_ar_tag.stl" scale="0.001 0.001 0.001"/>
+                    <mesh filename="package://interbotix_xsarm_descriptions/meshes/doris_arm_meshes/doris_arm_10_ar_tag.stl" />
                 </geometry>
                 <material name="interbotix_black"/>
@@ -298,5 +298,5 @@
                 <origin rpy="0 0 0" xyz="0 0 0"/>
                 <geometry>
-                    <mesh filename="package://interbotix_xsarm_descriptions/meshes/doris_arm_meshes/doris_arm_10_ar_tag.stl" scale="0.001 0.001 0.001"/>
+                    <mesh filename="package://interbotix_xsarm_descriptions/meshes/doris_arm_meshes/doris_arm_10_ar_tag.stl" />
                 </geometry>
             </collision>
@@ -320,5 +320,5 @@
                 <origin rpy="0 0 ${pi/2}" xyz="-0.063 0 0"/>
                 <geometry>
-                    <mesh filename="package://interbotix_xsarm_descriptions/meshes/doris_arm_meshes/doris_arm_8_gripper_bar.stl" scale="0.001 0.001 0.001"/>
+                    <mesh filename="package://interbotix_xsarm_descriptions/meshes/doris_arm_meshes/doris_arm_8_gripper_bar.stl" />
                 </geometry>
                 <material name="interbotix_black"/>
@@ -327,5 +327,5 @@
                 <origin rpy="0 0 ${pi/2}" xyz="-0.063 0 0"/>
                 <geometry>
-                    <mesh filename="package://interbotix_xsarm_descriptions/meshes/doris_arm_meshes/doris_arm_8_gripper_bar.stl" scale="0.001 0.001 0.001"/>
+                    <mesh filename="package://interbotix_xsarm_descriptions/meshes/doris_arm_meshes/doris_arm_8_gripper_bar.stl" />
                 </geometry>
             </collision-->
@@ -371,5 +371,5 @@
                     <origin rpy="${pi} 0 0" xyz="0 0 0"/>
                     <geometry>
-                        <mesh filename="package://interbotix_xsarm_descriptions/meshes/doris_arm_meshes/doris_arm_9_gripper_finger.stl" scale="0.001 0.001 0.001"/>
+                        <mesh filename="package://interbotix_xsarm_descriptions/meshes/doris_arm_meshes/doris_arm_9_gripper_finger.stl" />
                     </geometry>
                     <material name="interbotix_black"/>
@@ -378,5 +378,5 @@
                     <origin rpy="${pi} 0 0" xyz="0 0 0"/>
                     <geometry>
-                        <mesh filename="package://interbotix_xsarm_descriptions/meshes/doris_arm_meshes/doris_arm_9_gripper_finger.stl" scale="0.001 0.001 0.001"/>
+                        <mesh filename="package://interbotix_xsarm_descriptions/meshes/doris_arm_meshes/doris_arm_9_gripper_finger.stl" />
                     </geometry>
                 </collision>
@@ -411,5 +411,5 @@
                     <origin rpy="0 0 0" xyz="0 0 0 "/>
                     <geometry>
-                        <mesh filename="package://interbotix_xsarm_descriptions/meshes/doris_arm_meshes/doris_arm_9_gripper_finger.stl" scale="0.001 0.001 0.001"/>
+                        <mesh filename="package://interbotix_xsarm_descriptions/meshes/doris_arm_meshes/doris_arm_9_gripper_finger.stl" />
                     </geometry>
                     <material name="interbotix_black"/>
@@ -418,5 +418,5 @@
                     <origin rpy="0 0 0" xyz="0 0 0 "/>
                     <geometry>
-                        <mesh filename="package://interbotix_xsarm_descriptions/meshes/doris_arm_meshes/doris_arm_9_gripper_finger.stl" scale="0.001 0.001 0.001"/>
+                        <mesh filename="package://interbotix_xsarm_descriptions/meshes/doris_arm_meshes/doris_arm_9_gripper_finger.stl" />
                     </geometry>
                 </collision>

File: interbotix_ros_xsarms/interbotix_xsarm_moveit/config/srdf/doris_arm.srdf.xacro (robot description, xacro)
@@ -51,4 +51,11 @@
         <joint name="waist" value="0" />
         <joint name="wrist_angle" value="0.8" />
+        <joint name="wrist_rotate" value="0" />
+    </group_state>
+    <group_state name="Retreat" group="interbotix_arm">
+        <joint name="elbow" value="1.55" />
+        <joint name="shoulder" value="0" />
+        <joint name="waist" value="0" />
+        <joint name="wrist_angle" value="-0.7" />
         <joint name="wrist_rotate" value="0" />
     </group_state>

Commit message: reverting elbow

File: interbotix_ros_xsarms/interbotix_xsarm_descriptions/urdf/doris_arm.urdf.xacro (robot description, xacro)
@@ -84,5 +84,5 @@
     <joint name="shoulder" type="revolute">
         <axis xyz="0 1 0"/>
-        <limit effort="20" lower="${radians(-106)}" upper="${radians(72)}" velocity="${pi}"/>
+        <limit effort="20" lower="${radians(-106)}" upper="${radians(120)}" velocity="${pi}"/>
         <origin rpy="0 0 0" xyz="0 0 0.05805"/>
         <parent link="$(arg robot_name)/shoulder_link"/>
@@ -352,5 +352,5 @@
             <joint name="left_finger" type="prismatic">
                 <axis xyz="0 1 0"/>
-                <limit effort="5" lower="0.021" upper="0.057" velocity="1"/>
+                <limit effort="2" lower="0.014" upper="0.06145" velocity="1"/>
                 <origin rpy="0 0 0" xyz="0 0 0"/>
                 <parent link="$(arg robot_name)/fingers_link"/>
@@ -389,5 +389,5 @@
             <joint name="right_finger" type="prismatic">
                 <axis xyz="0 1 0"/>
-                <limit effort="5" lower="-0.057" upper="-0.021" velocity="1"/>
+                <limit effort="2" lower="-0.06145" upper="-0.014" velocity="1"/>
                 <origin rpy="0 0 0" xyz="0 0 0"/>
                 <parent link="$(arg robot_name)/fingers_link"/>

File: interbotix_ros_xsarms/interbotix_xsarm_moveit/config/srdf/doris_arm.srdf.xacro (robot description, xacro)
@@ -32,5 +32,5 @@
     </group>
     <!--GROUP STATES: Purpose: Define a named state for a particular group, in terms of joint values. This is useful to define states like 'folded arms'-->
-    <group_state name="Home" group="arm">
+    <group_state name="PrePick" group="arm">
         <joint name="elbow" value="1.3054176568984985" />
         <joint name="shoulder" value="-0.12271846830844879" />
@@ -38,4 +38,11 @@
         <joint name="wrist_angle" value="-1.4097284078598022" />
         <joint name="wrist_rotate" value="-0.030679617077112198" />
+    </group_state>
+    <group_state name="Home" group="arm">
+        <joint name="elbow" value="1.5493206977844238" />
+        <joint name="shoulder" value="-0.13499031960964203" />
+        <joint name="waist" value="-1.980369210243225" />
+        <joint name="wrist_angle" value="-1.5800002813339233" />
+        <joint name="wrist_rotate" value="-1.5999419689178467" />
     </group_state>
     <group_state name="Retreat" group="arm">
@@ -46,18 +53,32 @@
         <joint name="wrist_rotate" value="0" />
     </group_state>
-    <group_state name="Crane" group="arm">
+    <group_state name="CraneOld" group="arm">
         <joint name="elbow" value="0" />
         <joint name="shoulder" value="-0.004601942375302315" />
         <joint name="waist" value="0" />
         <joint name="wrist_angle" value="1.4" />
-        <joint name="wrist_rotate" value="0" />
+        <joint name="wrist_rotate" value="-1.57" />
+    </group_state>
+    <group_state name="Crane" group="arm">
+        <joint name="elbow" value="0.026077674701809883" />
+        <joint name="shoulder" value="0.8636311888694763" />
+        <joint name="waist" value="0" />
+        <joint name="wrist_angle" value="0.6826214790344238" />
+        <joint name="wrist_rotate" value="0.01840776950120926" />
+    </group_state>
+    <group_state name="GarbagePick" group="arm">
+        <joint name="elbow" value="-0.6703495979309082" />
+        <joint name="shoulder" value="1.7671458721160889" />
+        <joint name="waist" value="0" />
+        <joint name="wrist_angle" value="0.3466796576976776" />
+        <joint name="wrist_rotate" value="-0.003067961661145091" />
     </group_state>
     <group_state name="Closed" group="gripper">
-        <joint name="left_finger" value="0.021" />
-        <joint name="right_finger" value="-0.021" />
+        <joint name="left_finger" value="0.015" />
+        <joint name="right_finger" value="-0.015" />
     </group_state>
     <group_state name="Open" group="gripper">
-        <joint name="left_finger" value="0.057" />
-        <joint name="right_finger" value="-0.057" />
+        <joint name="left_finger" value="0.061" />
+        <joint name="right_finger" value="-0.061" />
     </group_state>
     <group_state name="Home" group="gripper">
