Commit message: :sparkles: feat: Implement new methods to control the arm

File: interbotix_ros_xsarms/interbotix_xsarm_descriptions/urdf/wx200.urdf.xacro (robot description, xacro)
@@ -1,4 +1,6 @@
 <?xml version="1.0"?>
 <robot name="wx200" xmlns:xacro="http://ros.org/wiki/xacro">
+<xacro:include filename="$(find doris_sensors_description)/urdf/realsense_camera.urdf.xacro" />
+    <xacro:include filename="$(find hector_sensors_description)/urdf/realsense_d435_camera.urdf.xacro" />
   <xacro:arg name="robot_name" default = "wx200"/>
   <xacro:arg name="base_link_frame" default="base_link"/>
@@ -24,4 +26,9 @@
     </joint>
   </xacro:if>
+  <xacro:realsense_camera name="camera" parent="world">
+    <!-- <link name="world"/> -->
+    <origin xyz="-0.34 0.0 0.465" rpy="0 0.26 0" />
+    <!-- <mesh filename="package://interbotix_xsarm_descriptions/meshes/realsense_d435_camera.dae"/> -->
+  </xacro:realsense_camera>
   <link name="$(arg robot_name)/$(arg base_link_frame)">
     <visual>

File: interbotix_ros_xsarms/interbotix_xsarm_moveit/config/srdf/wx200.srdf.xacro (robot description, xacro)
@@ -31,4 +31,5 @@
     </group>
     <!--GROUP STATES: Purpose: Define a named state for a particular group, in terms of joint values. This is useful to define states like 'folded arms'-->
+    <!-- ARM POSITIONS -->
     <group_state name="Home" group="interbotix_arm">
         <joint name="elbow" value="0" />
@@ -52,4 +53,13 @@
         <joint name="wrist_rotate" value="0" />
     </group_state>
+        <group_state name="PrePick" group="interbotix_arm">
+        <joint name="elbow" value="1.3023496866226196" />
+        <joint name="shoulder" value="-0.03221359848976135" />
+        <joint name="waist" value="-0.0015339808305725455" />
+        <joint name="wrist_angle" value="-1.3268934488296509" />
+        <joint name="wrist_rotate" value="0.07669904083013535" />
+    </group_state>
+    <!--  -->
+    <!-- GRIPPER POSITIONS -->
     <group_state name="Closed" group="interbotix_gripper">
         <joint name="left_finger" value="0.015" />
@@ -64,4 +74,5 @@
         <joint name="right_finger" value="-0.0195" />
     </group_state>
+    <!--  -->
     <!--END EFFECTOR: Purpose: Represent information about an end effector.-->
     <end_effector name="interbotix_gripper" parent_link="$(arg robot_name)/ee_gripper_link" group="interbotix_gripper" />

Commit message: came back to luis commit

File: interbotix_ros_xsarms/interbotix_xsarm_descriptions/urdf/wx200.urdf.xacro (robot description, xacro)
@@ -1,6 +1,5 @@
 <?xml version="1.0"?>
 <robot name="wx200" xmlns:xacro="http://ros.org/wiki/xacro">
-<xacro:include filename="$(find doris_sensors_description)/urdf/realsense_camera.urdf.xacro" />
-    <xacro:include filename="$(find hector_sensors_description)/urdf/realsense_d435_camera.urdf.xacro" />
+  <xacro:macro name="boris_arm" params="parent xyz rpy">
   <xacro:arg name="robot_name" default = "wx200"/>
   <xacro:arg name="base_link_frame" default="base_link"/>
@@ -26,9 +25,9 @@
     </joint>
   </xacro:if>
-  <xacro:realsense_camera name="camera" parent="world">
-    <!-- <link name="world"/> -->
-    <origin xyz="-0.34 0.0 0.465" rpy="0 0.26 0" />
-    <!-- <mesh filename="package://interbotix_xsarm_descriptions/meshes/realsense_d435_camera.dae"/> -->
-  </xacro:realsense_camera>
+  <joint name="arm_${parent}_joint" type="fixed">
+    <origin xyz="${xyz}" rpy="${rpy}"/>
+    <parent link="${parent}"/>
+    <child link="$(arg robot_name)/$(arg base_link_frame)"/>
+  </joint>
   <link name="$(arg robot_name)/$(arg base_link_frame)">
     <visual>
@@ -450,3 +449,4 @@
     <xacro:include filename="${urdf_loc}"/>
   </xacro:if>
+    </xacro:macro>
 </robot>

File: interbotix_ros_xsarms/interbotix_xsarm_moveit/config/srdf/wx200.srdf.xacro (robot description, xacro)
@@ -63,6 +63,6 @@
     <!-- GRIPPER POSITIONS -->
     <group_state name="Closed" group="interbotix_gripper">
-        <joint name="left_finger" value="0.015" />
-        <joint name="right_finger" value="-0.015" />
+        <joint name="left_finger" value="0.035" />
+        <joint name="right_finger" value="-0.035" />
     </group_state>
     <group_state name="Open" group="interbotix_gripper">

Commit message: :bug: Fix: Arm working with robot

File: interbotix_ros_xsarms/interbotix_xsarm_descriptions/urdf/wx200.urdf.xacro (robot description, xacro)
@@ -1,6 +1,5 @@
 <?xml version="1.0"?>
 <robot name="wx200" xmlns:xacro="http://ros.org/wiki/xacro">
-<xacro:include filename="$(find doris_sensors_description)/urdf/realsense_camera.urdf.xacro" />
-    <xacro:include filename="$(find hector_sensors_description)/urdf/realsense_d435_camera.urdf.xacro" />
+  <xacro:macro name="boris_arm" params="parent xyz rpy">
   <xacro:arg name="robot_name" default = "wx200"/>
   <xacro:arg name="base_link_frame" default="base_link"/>
@@ -26,9 +25,9 @@
     </joint>
   </xacro:if>
-  <xacro:realsense_camera name="camera" parent="world">
-    <!-- <link name="world"/> -->
-    <origin xyz="-0.34 0.0 0.465" rpy="0 0.26 0" />
-    <!-- <mesh filename="package://interbotix_xsarm_descriptions/meshes/realsense_d435_camera.dae"/> -->
-  </xacro:realsense_camera>
+  <joint name="arm_${parent}_joint" type="fixed">
+    <origin xyz="${xyz}" rpy="${rpy}"/>
+    <parent link="${parent}"/>
+    <child link="$(arg robot_name)/$(arg base_link_frame)"/>
+  </joint>
   <link name="$(arg robot_name)/$(arg base_link_frame)">
     <visual>
@@ -450,3 +449,4 @@
     <xacro:include filename="${urdf_loc}"/>
   </xacro:if>
+  </xacro:macro>
 </robot>
