Commit message: specific launch for doris arm moveit

File: interbotix_ros_xsarms/interbotix_xsarm_moveit/config/srdf/doris_arm.srdf.xacro (robot description, xacro)
@@ -16,5 +16,5 @@
     <xacro:arg name="external_srdf_loc" default=""/>
     <xacro:property name="srdf_loc" value="$(arg external_srdf_loc)"/>
-    <group name="interbotix_arm">
+    <group name="arm">
         <joint name="waist" />
         <joint name="shoulder" />
@@ -27,31 +27,17 @@
         <joint name="ee_gripper" />
     </group>
-    <group name="interbotix_gripper">
+    <group name="gripper">
         <link name="$(arg robot_name)/left_finger_link" />
         <link name="$(arg robot_name)/right_finger_link" />
     </group>
     <!--GROUP STATES: Purpose: Define a named state for a particular group, in terms of joint values. This is useful to define states like 'folded arms'-->
-    <group_state name="Home" group="interbotix_arm">
-        <joint name="elbow" value="0" />
-        <joint name="shoulder" value="0" />
+    <group_state name="Home" group="arm">
+        <joint name="elbow" value="1.3054176568984985" />
+        <joint name="shoulder" value="-0.12271846830844879" />
         <joint name="waist" value="0" />
-        <joint name="wrist_angle" value="0" />
-        <joint name="wrist_rotate" value="0" />
+        <joint name="wrist_angle" value="-1.4097284078598022" />
+        <joint name="wrist_rotate" value="-0.030679617077112198" />
     </group_state>
-    <group_state name="Upright" group="interbotix_arm">
-        <joint name="elbow" value="-1.5708" />
-        <joint name="shoulder" value="0" />
-        <joint name="waist" value="0" />
-        <joint name="wrist_angle" value="0" />
-        <joint name="wrist_rotate" value="0" />
-    </group_state>
-    <group_state name="Sleep" group="interbotix_arm">
-        <joint name="elbow" value="1.55" />
-        <joint name="shoulder" value="-1.76" />
-        <joint name="waist" value="0" />
-        <joint name="wrist_angle" value="0.8" />
-        <joint name="wrist_rotate" value="0" />
-    </group_state>
-    <group_state name="Retreat" group="interbotix_arm">
+    <group_state name="Retreat" group="arm">
         <joint name="elbow" value="1.55" />
         <joint name="shoulder" value="0" />
@@ -60,18 +46,25 @@
         <joint name="wrist_rotate" value="0" />
     </group_state>
-    <group_state name="Closed" group="interbotix_gripper">
+    <group_state name="Crane" group="arm">
+        <joint name="elbow" value="0" />
+        <joint name="shoulder" value="-0.004601942375302315" />
+        <joint name="waist" value="0" />
+        <joint name="wrist_angle" value="1.4" />
+        <joint name="wrist_rotate" value="0" />
+    </group_state>
+    <group_state name="Closed" group="gripper">
         <joint name="left_finger" value="0.021" />
         <joint name="right_finger" value="-0.021" />
     </group_state>
-    <group_state name="Open" group="interbotix_gripper">
+    <group_state name="Open" group="gripper">
         <joint name="left_finger" value="0.057" />
         <joint name="right_finger" value="-0.057" />
     </group_state>
-    <group_state name="Home" group="interbotix_gripper">
+    <group_state name="Home" group="gripper">
         <joint name="left_finger" value="0.03" />
         <joint name="right_finger" value="-0.03" />
     </group_state>
     <!--END EFFECTOR: Purpose: Represent information about an end effector.-->
-    <end_effector name="interbotix_gripper" parent_link="$(arg robot_name)/ee_gripper_link" group="interbotix_gripper" />
+    <end_effector name="gripper" parent_link="$(arg robot_name)/ee_gripper_link" group="gripper" />
     <!--DISABLE COLLISIONS: By default it is assumed that any link of the robot could potentially come into collision with any other link in the robot. This tag disables collision checking between a specified pair of links. -->
     <disable_collisions link1="$(arg robot_name)/$(arg base_link_frame)" link2="$(arg robot_name)/shoulder_link" reason="Adjacent" />

Commit message: added carry my luggage pose

File: interbotix_ros_xsarms/interbotix_xsarm_moveit/config/srdf/doris_arm.srdf.xacro (robot description, xacro)
@@ -74,4 +74,11 @@
         <joint name="wrist_rotate" value="-0.003067961661145091" />
     </group_state>
+    <group_state name="BagHook" group="arm">
+        <joint name="elbow" value="1.0078253746032715" />
+        <joint name="shoulder" value="-0.18561168015003204" />
+        <joint name="waist" value="-0.02454369328916073" />
+        <joint name="wrist_angle" value="-1.5416507720947266" />
+        <joint name="wrist_rotate" value="-1.5907381772994995" />
+    </group_state>
     <group_state name="Closed" group="gripper">
         <joint name="left_finger" value="0.015" />

Commit message: adding cranehigh pose

File: interbotix_ros_xsarms/interbotix_xsarm_moveit/config/srdf/doris_arm.srdf.xacro (robot description, xacro)
@@ -53,10 +53,10 @@
         <joint name="wrist_rotate" value="0" />
     </group_state>
-    <group_state name="CraneOld" group="arm">
-        <joint name="elbow" value="0" />
-        <joint name="shoulder" value="-0.004601942375302315" />
-        <joint name="waist" value="0" />
-        <joint name="wrist_angle" value="1.4" />
-        <joint name="wrist_rotate" value="-1.57" />
+    <group_state name="CraneHigh" group="arm">
+        <joint name="elbow" value="0.0" />
+        <joint name="shoulder" value="0.25003886222839355" />
+        <joint name="waist" value="-0.04908738657832146" />
+        <joint name="wrist_angle" value="1.2701361179351807" />
+        <joint name="wrist_rotate" value="0.016873789951205254" />
     </group_state>
     <group_state name="Crane" group="arm">

Commit message: gripper update working

File: interbotix_ros_xsarms/interbotix_xsarm_moveit/config/srdf/doris_arm.srdf.xacro (robot description, xacro)
@@ -41,22 +41,29 @@
     <group_state name="Home" group="arm">
         <joint name="elbow" value="1.5493206977844238" />
-        <joint name="shoulder" value="-0.13499031960964203" />
-        <joint name="waist" value="-1.980369210243225" />
-        <joint name="wrist_angle" value="-1.5800002813339233" />
-        <joint name="wrist_rotate" value="-1.5999419689178467" />
+        <joint name="shoulder" value="0.0" />
+        <joint name="waist" value="-1.5707963267948966" />
+        <joint name="wrist_angle" value="-1.716524600982666" />
+        <joint name="wrist_rotate" value="1.6275537014007568" />
     </group_state>
     <group_state name="Retreat" group="arm">
-        <joint name="elbow" value="1.55" />
-        <joint name="shoulder" value="0" />
-        <joint name="waist" value="0" />
-        <joint name="wrist_angle" value="-0.7" />
-        <joint name="wrist_rotate" value="0" />
+        <joint name="elbow" value="1.667437195777893" />
+        <joint name="shoulder" value="-0.2684466540813446" />
+        <joint name="waist" value="-2.0678062438964844" />
+        <joint name="wrist_angle" value="-1.6428934335708618" />
+        <joint name="wrist_rotate" value="1.543184757232666" />
+    </group_state>
+        <group_state name="RetreatEmilly" group="arm">
+        <joint name="elbow" value="1.6106798648834229" />
+        <joint name="shoulder" value="-0.2684466540813446" />
+        <joint name="waist" value="-1.9819031953811646" />
+        <joint name="wrist_angle" value="-1.5846022367477417" />
+        <joint name="wrist_rotate" value="-0.023009711876511574" />
     </group_state>
     <group_state name="CraneHigh" group="arm">
-        <joint name="elbow" value="0.0" />
-        <joint name="shoulder" value="0.25003886222839355" />
-        <joint name="waist" value="-0.04908738657832146" />
-        <joint name="wrist_angle" value="1.2701361179351807" />
-        <joint name="wrist_rotate" value="0.016873789951205254" />
+        <joint name="elbow" value="0.11811652034521103" />
+        <joint name="shoulder" value="0.475534051656723" />
+        <joint name="waist" value="0.003067961661145091" />
+        <joint name="wrist_angle" value="0.872835099697113" />
+        <joint name="wrist_rotate" value="0.04295146465301514" />
     </group_state>
     <group_state name="Crane" group="arm">
@@ -66,4 +73,32 @@
         <joint name="wrist_angle" value="0.6826214790344238" />
         <joint name="wrist_rotate" value="0.01840776950120926" />
+    </group_state>
+        <group_state name="Pick" group="arm">
+        <joint name="elbow" value="0.5675728917121887" />
+        <joint name="shoulder" value="1.0937283039093018" />
+        <joint name="waist" value="0.07056311517953873" />
+        <joint name="wrist_angle" value="0.11965050548315048" />
+        <joint name="wrist_rotate" value="1.494097352027893" />
+    </group_state>
+    <group_state name="PickUp" group="arm">
+        <joint name="elbow" value="0.3988350033760071" />
+        <joint name="shoulder" value="1.3192235231399536" />
+        <joint name="waist" value="0.0782330259680748" />
+        <joint name="wrist_angle" value="0.10277671366930008" />
+        <joint name="wrist_rotate" value="1.4864274263381958" />
+    </group_state>
+        <group_state name="PickBack" group="arm">
+        <joint name="elbow" value="0.026077674701809883" />
+        <joint name="shoulder" value="1.5155730247497559" />
+        <joint name="waist" value="0.01840776950120926" />
+        <joint name="wrist_angle" value="-1.716524600982666" />
+        <joint name="wrist_rotate" value="1.6275537014007568" />
+    </group_state>
+        <group_state name="PrePickBack" group="arm">
+        <joint name="elbow" value="1.3054176568984985" />
+        <joint name="shoulder" value="-0.12271846830844879" />
+        <joint name="waist" value="0" />
+        <joint name="wrist_angle" value="-1.716524600982666" />
+        <joint name="wrist_rotate" value="1.6275537014007568" />
     </group_state>
     <group_state name="GarbagePick" group="arm">
@@ -80,4 +115,15 @@
         <joint name="wrist_angle" value="-1.5416507720947266" />
         <joint name="wrist_rotate" value="-1.5907381772994995" />
+    </group_state>
+    <group_state name="BagNav" group="arm">
+        <joint name="elbow" value="1.3360973596572876" />
+        <joint name="shoulder" value="-0.11198060214519501" />
+        <joint name="waist" value="0.05062136799097061" />
+        <joint name="wrist_angle" value="-1.6873788833618164" />
+        <joint name="wrist_rotate" value="-1.6352235078811646" />
+    </group_state>
+    <group_state name="BagGripper" group="gripper">
+        <joint name="left_finger" value="0.020" />
+        <joint name="right_finger" value="-0.020" />
     </group_state>
     <group_state name="Closed" group="gripper">

Commit message: new arm positions for take out the garbage

File: interbotix_ros_xsarms/interbotix_xsarm_moveit/config/srdf/doris_arm.srdf.xacro (robot description, xacro)
@@ -46,4 +46,11 @@
         <joint name="wrist_rotate" value="1.6275537014007568" />
     </group_state>
+    <group_state name="NewScissorsHome" group="arm">
+        <joint name="elbow" value="1.5493206977844238" />
+        <joint name="shoulder" value="0.0" />
+        <joint name="waist" value="-1.5707963267948966" />
+        <joint name="wrist_angle" value="-1.6643692255020142" />
+        <joint name="wrist_rotate" value="-0.026077674701809883" />
+    </group_state>
     <group_state name="Retreat" group="arm">
         <joint name="elbow" value="1.667437195777893" />
@@ -122,4 +129,18 @@
         <joint name="wrist_angle" value="-1.6873788833618164" />
         <joint name="wrist_rotate" value="-1.6352235078811646" />
+    </group_state>
+        <group_state name="NewGarbagePick" group="arm">
+        <joint name="elbow" value="0.8375535607337952" />
+        <joint name="shoulder" value="0.7194370031356812" />
+        <joint name="waist" value="-0.00920388475060463" />
+        <joint name="wrist_angle" value="0.12118448317050934" />
+        <joint name="wrist_rotate" value="0.05368933081626892" />
+    </group_state>
+    <group_state name="NewGarbagePickUp" group="arm">
+        <joint name="elbow" value="0.03221359848976135" />
+        <joint name="shoulder" value="1.6613012552261353" />
+        <joint name="waist" value="-0.05675728991627693" />
+        <joint name="wrist_angle" value="0.12118448317050934" />
+        <joint name="wrist_rotate" value="0.05368933081626892" />
     </group_state>
     <group_state name="BagGripper" group="gripper">

Commit message: arm tests

File: interbotix_ros_xsarms/interbotix_xsarm_moveit/config/srdf/doris_arm.srdf.xacro (robot description, xacro)
@@ -131,16 +131,16 @@
     </group_state>
         <group_state name="NewGarbagePick" group="arm">
-        <joint name="elbow" value="0.8375535607337952" />
-        <joint name="shoulder" value="0.7194370031356812" />
-        <joint name="waist" value="-0.00920388475060463" />
-        <joint name="wrist_angle" value="0.12118448317050934" />
-        <joint name="wrist_rotate" value="0.05368933081626892" />
+        <joint name="elbow" value="0.5921165943145752" />
+        <joint name="shoulder" value="1.1060001850128174" />
+        <joint name="waist" value="0.0" />
+        <joint name="wrist_angle" value="0.11965050548315048" />
+        <joint name="wrist_rotate" value="1.494097352027893" />
     </group_state>
     <group_state name="NewGarbagePickUp" group="arm">
         <joint name="elbow" value="0.03221359848976135" />
         <joint name="shoulder" value="1.6613012552261353" />
-        <joint name="waist" value="-0.05675728991627693" />
-        <joint name="wrist_angle" value="0.12118448317050934" />
-        <joint name="wrist_rotate" value="0.05368933081626892" />
+        <joint name="waist" value="0.0" />
+        <joint name="wrist_angle" value="0.11965050548315048" />
+        <joint name="wrist_rotate" value="1.494097352027893" />
     </group_state>
     <group_state name="BagGripper" group="gripper">

Commit message: tava no robo

File: interbotix_ros_xsarms/interbotix_xsarm_moveit/config/srdf/doris_arm.srdf.xacro (robot description, xacro)
@@ -47,9 +47,9 @@
     </group_state>
     <group_state name="NewScissorsHome" group="arm">
-        <joint name="elbow" value="1.5493206977844238" />
-        <joint name="shoulder" value="0.0" />
-        <joint name="waist" value="-1.5707963267948966" />
-        <joint name="wrist_angle" value="-1.6643692255020142" />
-        <joint name="wrist_rotate" value="-0.026077674701809883" />
+        <joint name="elbow" value="1.5984079837799072" />
+        <joint name="shoulder" value="-0.1257864236831665" />
+        <joint name="waist" value="1.555456519126892" />
+        <joint name="wrist_angle" value="-1.6735731363296509" />
+        <joint name="wrist_rotate" value="-0.07516506314277649" />
     </group_state>
     <group_state name="Retreat" group="arm">

Commit message: tava no robo

File: interbotix_ros_xsarms/interbotix_xsarm_moveit/config/srdf/doris_arm.srdf.xacro (robot description, xacro)
@@ -38,4 +38,11 @@
         <joint name="wrist_angle" value="-1.4097284078598022" />
         <joint name="wrist_rotate" value="-0.030679617077112198" />
+    </group_state>
+    <group_state name="PrePickGarbage" group="arm">
+        <joint name="elbow" value="1.3054176568984985" />
+        <joint name="shoulder" value="-0.12271846830844879" />
+        <joint name="waist" value="0" />
+        <joint name="wrist_angle" value="-1.4097284078598022" />
+        <joint name="wrist_rotate" value="1.494097352027893" />
     </group_state>
     <group_state name="Home" group="arm">

Commit message: new arm positions

File: interbotix_ros_xsarms/interbotix_xsarm_moveit/config/srdf/doris_arm.srdf.xacro (robot description, xacro)
@@ -46,4 +46,11 @@
         <joint name="wrist_rotate" value="1.494097352027893" />
     </group_state>
+    <group_state name="DropGarbage" group="arm">
+        <joint name="elbow" value="1.3176895380020142" />
+        <joint name="shoulder" value="-0.08283496648073196" />
+        <joint name="waist" value="0" />
+        <joint name="wrist_angle" value="0.27458256483078003" />
+        <joint name="wrist_rotate" value="1.5968739986419678" />
+    </group_state>
     <group_state name="Home" group="arm">
         <joint name="elbow" value="1.5493206977844238" />
@@ -52,11 +59,4 @@
         <joint name="wrist_angle" value="-1.716524600982666" />
         <joint name="wrist_rotate" value="1.6275537014007568" />
-    </group_state>
-    <group_state name="NewScissorsHome" group="arm">
-        <joint name="elbow" value="1.5984079837799072" />
-        <joint name="shoulder" value="-0.1257864236831665" />
-        <joint name="waist" value="1.555456519126892" />
-        <joint name="wrist_angle" value="-1.6735731363296509" />
-        <joint name="wrist_rotate" value="-0.07516506314277649" />
     </group_state>
     <group_state name="Retreat" group="arm">
@@ -116,11 +116,4 @@
         <joint name="wrist_rotate" value="1.6275537014007568" />
     </group_state>
-    <group_state name="GarbagePick" group="arm">
-        <joint name="elbow" value="-0.6703495979309082" />
-        <joint name="shoulder" value="1.7671458721160889" />
-        <joint name="waist" value="0" />
-        <joint name="wrist_angle" value="0.3466796576976776" />
-        <joint name="wrist_rotate" value="-0.003067961661145091" />
-    </group_state>
     <group_state name="BagHook" group="arm">
         <joint name="elbow" value="1.0078253746032715" />
@@ -137,17 +130,10 @@
         <joint name="wrist_rotate" value="-1.6352235078811646" />
     </group_state>
-        <group_state name="NewGarbagePick" group="arm">
-        <joint name="elbow" value="0.5921165943145752" />
-        <joint name="shoulder" value="1.1060001850128174" />
+        <group_state name="GarbagePick" group="arm">
+        <joint name="elbow" value="0.9740778207778931" />
+        <joint name="shoulder" value="0.6718835830688477" />
         <joint name="waist" value="0.0" />
-        <joint name="wrist_angle" value="0.11965050548315048" />
-        <joint name="wrist_rotate" value="1.494097352027893" />
-    </group_state>
-    <group_state name="NewGarbagePickUp" group="arm">
-        <joint name="elbow" value="0.03221359848976135" />
-        <joint name="shoulder" value="1.6613012552261353" />
-        <joint name="waist" value="0.0" />
-        <joint name="wrist_angle" value="0.11965050548315048" />
-        <joint name="wrist_rotate" value="1.494097352027893" />
+        <joint name="wrist_angle" value="-0.004601942375302315" />
+        <joint name="wrist_rotate" value="1.5646604299545288" />
     </group_state>
     <group_state name="BagGripper" group="gripper">

Commit message: release_1 pose

File: interbotix_ros_xsarms/interbotix_xsarm_moveit/config/srdf/doris_arm.srdf.xacro (robot description, xacro)
@@ -139,4 +139,11 @@
         <joint name="right_finger" value="-0.03" />
     </group_state>
+    <group_state name="release_1" group="arm">
+        <joint name="elbow" value="-0.3911651074886322" />
+        <joint name="shoulder" value="0.7225049734115601" />
+        <joint name="waist" value="-0.200951486825943" />
+        <joint name="wrist_angle" value="-0.3911651074886322" />
+        <joint name="wrist_rotate" value="-0.04601942375302315" />
+    </group_state>
     <!--END EFFECTOR: Purpose: Represent information about an end effector.-->
     <end_effector name="gripper" parent_link="$(arg robot_name)/ee_gripper_link" group="gripper" />

Commit message: added new poses, HomeLeft and RetreatLeft

File: interbotix_ros_xsarms/interbotix_xsarm_moveit/config/srdf/doris_arm.srdf.xacro (robot description, xacro)
@@ -58,4 +58,11 @@
         <joint name="waist" value="-1.5707963267948966" />
         <joint name="wrist_angle" value="-1.716524600982666" />
+        <joint name="wrist_rotate" value="1.5339808464050293" />
+    </group_state>
+    <group_state name="HomeLeft" group="arm">
+        <joint name="elbow" value="1.6290876865386963" />
+        <joint name="shoulder" value="0.0" />
+        <joint name="waist" value="1.575398325920105" />
+        <joint name="wrist_angle" value="-1.6965827941894531" />
         <joint name="wrist_rotate" value="1.6275537014007568" />
     </group_state>
@@ -67,10 +74,10 @@
         <joint name="wrist_rotate" value="1.543184757232666" />
     </group_state>
-        <group_state name="RetreatEmilly" group="arm">
-        <joint name="elbow" value="1.6106798648834229" />
-        <joint name="shoulder" value="-0.2684466540813446" />
-        <joint name="waist" value="-1.9819031953811646" />
-        <joint name="wrist_angle" value="-1.5846022367477417" />
-        <joint name="wrist_rotate" value="-0.023009711876511574" />
+        <group_state name="RetreatLeft" group="arm">
+        <joint name="elbow" value="1.656699299812317" />
+        <joint name="shoulder" value="-0.28941750168800354" />
+        <joint name="waist" value="2.0540003776550293" />
+        <joint name="wrist_angle" value="-1.6904468536376953" />
+        <joint name="wrist_rotate" value="1.5569905042648315" />
     </group_state>
     <group_state name="CraneHigh" group="arm">

Commit message: pre release pose

File: interbotix_ros_xsarms/interbotix_xsarm_moveit/config/srdf/doris_arm.srdf.xacro (robot description, xacro)
@@ -146,4 +146,11 @@
         <joint name="wrist_rotate" value="-0.04601942375302315" />
     </group_state>
+        <group_state name="pre_release" group="arm">
+        <joint name="elbow" value="0.16106799244880676" />
+        <joint name="shoulder" value="-0.06596117466688156" />
+        <joint name="waist" value="-0.04295146465301514" />
+        <joint name="wrist_angle" value="0.05368933081626892" />
+        <joint name="wrist_rotate" value="-0.03681553900241852" />
+    </group_state>
     <!--END EFFECTOR: Purpose: Represent information about an end effector.-->
     <end_effector name="gripper" parent_link="$(arg robot_name)/ee_gripper_link" group="gripper" />
