Commit message: fixed some arm poses, added 0.0 to waist

File: interbotix_ros_xsarms/interbotix_xsarm_moveit/config/srdf/doris_arm.srdf.xacro (robot description, xacro)
@@ -98,5 +98,5 @@
         <joint name="elbow" value="0.5675728917121887" />
         <joint name="shoulder" value="1.0937283039093018" />
-        <joint name="waist" value="0.07056311517953873" />
+        <joint name="waist" value="0.0" />
         <joint name="wrist_angle" value="0.11965050548315048" />
         <joint name="wrist_rotate" value="1.494097352027893" />
@@ -105,5 +105,5 @@
         <joint name="elbow" value="0.3988350033760071" />
         <joint name="shoulder" value="1.3192235231399536" />
-        <joint name="waist" value="0.0782330259680748" />
+        <joint name="waist" value="0.0" />
         <joint name="wrist_angle" value="0.10277671366930008" />
         <joint name="wrist_rotate" value="1.4864274263381958" />
@@ -112,5 +112,5 @@
         <joint name="elbow" value="0.026077674701809883" />
         <joint name="shoulder" value="1.5155730247497559" />
-        <joint name="waist" value="0.01840776950120926" />
+        <joint name="waist" value="0.0" />
         <joint name="wrist_angle" value="-1.716524600982666" />
         <joint name="wrist_rotate" value="1.6275537014007568" />
@@ -119,5 +119,5 @@
         <joint name="elbow" value="1.3054176568984985" />
         <joint name="shoulder" value="-0.12271846830844879" />
-        <joint name="waist" value="0" />
+        <joint name="waist" value="0.0" />
         <joint name="wrist_angle" value="-1.716524600982666" />
         <joint name="wrist_rotate" value="1.6275537014007568" />
@@ -127,6 +127,6 @@
         <joint name="shoulder" value="-0.18561168015003204" />
         <joint name="waist" value="-0.02454369328916073" />
-        <joint name="wrist_angle" value="-1.5416507720947266" />
-        <joint name="wrist_rotate" value="-1.5907381772994995" />
+        <joint name="wrist_angle" value="-1.6965827941894531" />
+        <joint name="wrist_rotate" value="1.5569905042648315" />
     </group_state>
     <group_state name="BagNav" group="arm">

Commit message: MANIPULATION - save new home pose to manipulation

File: interbotix_ros_xsarms/interbotix_xsarm_moveit/config/srdf/doris_arm.srdf.xacro (robot description, xacro)
@@ -146,5 +146,5 @@
         <joint name="wrist_rotate" value="-0.04601942375302315" />
     </group_state>
-        <group_state name="pre_release" group="arm">
+    <group_state name="pre_release" group="arm">
         <joint name="elbow" value="0.16106799244880676" />
         <joint name="shoulder" value="-0.06596117466688156" />
@@ -152,4 +152,11 @@
         <joint name="wrist_angle" value="0.05368933081626892" />
         <joint name="wrist_rotate" value="-0.03681553900241852" />
+    </group_state>
+    <group_state name="Home_manipulation" group="arm">
+        <joint name="elbow" value="1.3115535974502563" />
+        <joint name="shoulder" value="0.4049709439277649" />
+        <joint name="waist" value="1.8637866973876953," />
+        <joint name="wrist_angle" value="0.04908738657832146" />
+        <joint name="wrist_rotate" value="0.07976700365543365" />
     </group_state>
     <!--END EFFECTOR: Purpose: Represent information about an end effector.-->

Commit message: {MANIPULATION} - Update Home_release waist value

File: interbotix_ros_xsarms/interbotix_xsarm_moveit/config/srdf/doris_arm.srdf.xacro (robot description, xacro)
@@ -156,5 +156,5 @@
         <joint name="elbow" value="1.3115535974502563" />
         <joint name="shoulder" value="0.4049709439277649" />
-        <joint name="waist" value="1.8637866973876953," />
+        <joint name="waist" value="1.8637866973876953" />
         <joint name="wrist_angle" value="0.04908738657832146" />
         <joint name="wrist_rotate" value="0.07976700365543365" />

Commit message: new pose to carry two bags

File: interbotix_ros_xsarms/interbotix_xsarm_moveit/config/srdf/doris_arm.srdf.xacro (robot description, xacro)
@@ -45,4 +45,11 @@
         <joint name="wrist_angle" value="-1.4097284078598022" />
         <joint name="wrist_rotate" value="1.494097352027893" />
+    </group_state>
+    <group_state name="ReleaseBag" group="arm">
+        <joint name="elbow" value="0.6504078507423401" />
+        <joint name="shoulder" value="-0.3911651074886322" />
+        <joint name="waist" value="1.8361750841140747" />
+        <joint name="wrist_angle" value="1.5477867126464844" />
+        <joint name="wrist_rotate" value="1.6520973443984985" />
     </group_state>
     <group_state name="DropGarbage" group="arm">

Commit message: new pose to mor

File: interbotix_ros_xsarms/interbotix_xsarm_moveit/config/srdf/doris_arm.srdf.xacro (robot description, xacro)
@@ -159,4 +159,11 @@
         <joint name="wrist_angle" value="0.04908738657832146" />
         <joint name="wrist_rotate" value="0.07976700365543365" />
+    </group_state>
+    <group_state name="Pre_Release_manipulation" group="arm">
+        <joint name="elbow" value="0.9142525792121887" />
+        <joint name="shoulder" value="0.780796229839325" />
+        <joint name="waist" value="-0.016873789951205254" />
+        <joint name="wrist_angle" value="-1.6474953889846802" />
+        <joint name="wrist_rotate" value="0.07516506314277649" />
     </group_state>
     <!--END EFFECTOR: Purpose: Represent information about an end effector.-->
