Commit message: modifications for gpsr

File: interbotix_ros_xsarms/interbotix_xsarm_moveit/config/srdf/vx300s.srdf.xacro (robot description, xacro)
@@ -37,5 +37,5 @@
         <joint name="shoulder" value="0" />
         <joint name="waist" value="0" />
-        <joint name="wrist_angle" value="0" />
+        <joint name="wrist_angle" value="1.5708" />
         <joint name="wrist_rotate" value="0" />
     </group_state>
