Commit message: :sparkles: New gripper config

File: interbotix_ros_xsarms/interbotix_xsarm_moveit/config/srdf/wx200.srdf.xacro (robot description, xacro)
@@ -67,6 +67,6 @@
     </group_state>
     <group_state name="Open" group="interbotix_gripper">
-        <joint name="left_finger" value="0.037" />
-        <joint name="right_finger" value="-0.037" />
+        <joint name="left_finger" value="0.032" />
+        <joint name="right_finger" value="-0.032" />
     </group_state>
     <group_state name="Home" group="interbotix_gripper">
